Commit message: robot's model is seen both rviz and gazebo

File: install/set_slam/share/set_slam/urdf/acrome_mini_robot.xacro (robot description, xacro)
@@ -19,5 +19,5 @@
       <origin xyz="0 0 0" rpy="0 0 0"/>
       <geometry>
-        <mesh filename="$(arg mesh_path)/base_link.stl" scale="1 1 1"/>
+        <mesh filename="file:///home/halit/acrome_mini_robot/src/set_slam/meshes/base_link.stl" scale="1 1 1"/>
       </geometry>
       <material name="base_grey">
@@ -28,5 +28,5 @@
       <origin xyz="0 0 0" rpy="0 0 0"/>
       <geometry>
-        <mesh filename="$(arg mesh_path)/base_link.stl" scale="1 1 1"/>
+        <mesh filename="file:///home/halit/acrome_mini_robot/src/set_slam/meshes/base_link.stl" scale="1 1 1"/>
       </geometry>
     </collision>
@@ -50,5 +50,5 @@
       <origin xyz="0 0 0" rpy="0 0 0"/>
       <geometry>
-        <mesh filename="$(arg mesh_path)/left_wheel.stl" scale="1 1 1"/>
+        <mesh filename="file:///home/halit/acrome_mini_robot/src/set_slam/meshes/left_wheel.stl" scale="1 1 1"/>
       </geometry>
       <material name="wheel_black">
@@ -59,5 +59,5 @@
       <origin xyz="0 0 0" rpy="0 0 0"/>
       <geometry>
-        <mesh filename="$(arg mesh_path)/left_wheel.stl" scale="1 1 1"/>
+        <mesh filename="file:///home/halit/acrome_mini_robot/src/set_slam/meshes/left_wheel.stl" scale="1 1 1"/>
       </geometry>
     </collision>
@@ -84,5 +84,5 @@
       <origin xyz="0 0 0" rpy="0 0 0"/>
       <geometry>
-        <mesh filename="$(arg mesh_path)/right_wheel.stl" scale="1 1 1"/>
+        <mesh filename="file:///home/halit/acrome_mini_robot/src/set_slam/meshes/right_wheel.stl" scale="1 1 1"/>
       </geometry>
       <material name="wheel_black"/>
@@ -91,5 +91,5 @@
       <origin xyz="0 0 0" rpy="0 0 0"/>
       <geometry>
-        <mesh filename="$(arg mesh_path)/right_wheel.stl" scale="1 1 1"/>
+        <mesh filename="file:///home/halit/acrome_mini_robot/src/set_slam/meshes/right_wheel.stl" scale="1 1 1"/>
       </geometry>
     </collision>

Commit message: developed teleop app and created ground world

File: install/set_slam/share/set_slam/urdf/acrome_mini_robot.xacro (robot description, xacro)
@@ -1,138 +1,232 @@
 <?xml version="1.0"?>
 <robot name="acrome_mini_robot" xmlns:xacro="http://www.ros.org/wiki/xacro">
-  <!-- #############################################
-       Minimal differential-drive URDF using STL meshes
-       Paths are absolute as provided by you. Adjust joint/origin xyz
-       values if the wheels do not align perfectly with the base mesh.
-       REP-103 frames: +X forward, +Y left, +Z up.
-       ############################################# -->
-  <!-- ================= Base Link ================= -->
+  <!-- Parametreler -->
+  <xacro:property name="PI" value="3.141592653589793"/>
+  <!-- Ana robot gövdesi -->
   <link name="base_link">
-    <inertial>
-      <!-- Placeholder inertia; replace with measured values if available -->
-      <origin xyz="0 0 0" rpy="0 0 0"/>
-      <mass value="2.0"/>
-      <inertia ixx="0.02" ixy="0.0" ixz="0.0" iyy="0.03" iyz="0.0" izz="0.03"/>
-    </inertial>
-    <visual>
-      <!-- If the model looks flipped, try rpy="0 0 3.14159" -->
-      <origin xyz="0 0 0" rpy="0 0 0"/>
+    <visual>
       <geometry>
         <mesh filename="file:///home/halit/acrome_mini_robot/src/set_slam/meshes/base_link.stl" scale="1 1 1"/>
       </geometry>
-      <material name="base_grey">
-        <color rgba="0.6 0.6 0.6 1.0"/>
-      </material>
-    </visual>
-    <collision>
-      <origin xyz="0 0 0" rpy="0 0 0"/>
-      <geometry>
-        <mesh filename="file:///home/halit/acrome_mini_robot/src/set_slam/meshes/base_link.stl" scale="1 1 1"/>
-      </geometry>
-    </collision>
-  </link>
-  <!-- A flat frame on the ground projection of base_link (handy for navigation) -->
-  <link name="base_footprint"/>
-  <joint name="base_footprint_joint" type="fixed">
-    <parent link="base_footprint"/>
-    <child link="base_link"/>
-    <!-- Set z so base_footprint sits on the ground if your base_link z-origin is above ground -->
-    <origin xyz="0 0 0" rpy="0 0 0"/>
-  </joint>
-  <!-- ================ Left Wheel ================ -->
-  <link name="left_wheel_link">
-    <inertial>
-      <origin xyz="0 0 0" rpy="0 0 0"/>
+      <origin xyz="0 0 0.075" rpy="0 0 -1.5708"/>
+      <material name="blue">
+        <color rgba="0.2 0.2 0.8 1"/>
+      </material>
+    </visual>
+    <collision>
+      <geometry>
+        <cylinder radius="0.25" length="0.15"/>
+      </geometry>
+      <origin xyz="0 0 0.075" rpy="0 0 -1.5708"/>
+    </collision>
+    <inertial>
+      <mass value="5.0"/>
+      <origin xyz="0 0 0.075" rpy="0 0 0"/>
+      <inertia ixx="0.2083" ixy="0.0" ixz="0.0" iyy="0.2083" iyz="0.0" izz="0.3125"/>
+    </inertial>
+  </link>
+  <!-- Caster Wheel Support (Destek Çubuğu) -->
+  <link name="caster_support">
+    <visual>
+      <geometry>
+        <cylinder radius="0.005" length="0.03"/>
+      </geometry>
+      <origin xyz="0 0 -0.015" rpy="0 0 0"/>
+      <material name="gray">
+        <color rgba="0.5 0.5 0.5 1"/>
+      </material>
+    </visual>
+    <collision>
+      <geometry>
+        <cylinder radius="0.005" length="0.03"/>
+      </geometry>
+      <origin xyz="0 0 -0.015" rpy="0 0 0"/>
+    </collision>
+    <inertial>
+      <mass value="0.05"/>
+      <origin xyz="0 0 -0.015" rpy="0 0 0"/>
+      <inertia ixx="0.00001" ixy="0" ixz="0" iyy="0.00001" iyz="0" izz="0.00001"/>
+    </inertial>
+  </link>
+  <!-- Caster Wheel -->
+  <link name="caster_wheel">
+    <visual>
+      <geometry>
+        <sphere radius="0.02"/>
+      </geometry>
+      <origin xyz="0 0 0" rpy="0 0 0"/>
+      <material name="black">
+        <color rgba="0.1 0.1 0.1 1"/>
+      </material>
+    </visual>
+    <collision>
+      <geometry>
+        <sphere radius="0.02"/>
+      </geometry>
+      <origin xyz="0 0 0" rpy="0 0 0"/>
+    </collision>
+    <inertial>
+      <mass value="0.1"/>
+      <origin xyz="0 0 0" rpy="0 0 0"/>
+      <inertia ixx="0.000016" ixy="0" ixz="0" iyy="0.000016" iyz="0" izz="0.000016"/>
+    </inertial>
+  </link>
+  <!-- Tekerlek 2 -->
+  <link name="wheel_2">
+    <visual>
+      <geometry>
+        <mesh filename="file:///home/halit/acrome_mini_robot/src/set_slam/meshes/left_wheel.stl" scale="0.7 0.7 0.7"/>
+      </geometry>
+      <origin xyz="0 0 0" rpy="1.5708 0 0"/>
+      <material name="black">
+        <color rgba="0.1 0.1 0.1 1"/>
+      </material>
+    </visual>
+    <collision>
+      <surface>
+        <friction>
+          <ode>
+            <mu>1.0</mu>
+            <mu2>1.0</mu2>
+          </ode>
+        </friction>
+      </surface>
+      <geometry>
+        <cylinder radius="0.06" length="0.025"/>
+      </geometry>
+      <origin xyz="0 0 0" rpy="1.5708 0 0"/>
+    </collision>
+    <inertial>
       <mass value="0.25"/>
-      <inertia ixx="0.0005" ixy="0.0" ixz="0.0" iyy="0.0007" iyz="0.0" izz="0.0005"/>
-    </inertial>
-    <visual>
-      <origin xyz="0 0 0" rpy="0 0 0"/>
-      <geometry>
-        <mesh filename="file:///home/halit/acrome_mini_robot/src/set_slam/meshes/left_wheel.stl" scale="1 1 1"/>
-      </geometry>
-      <material name="wheel_black">
-        <color rgba="0.1 0.1 0.1 1.0"/>
-      </material>
-    </visual>
-    <collision>
-      <origin xyz="0 0 0" rpy="0 0 0"/>
-      <geometry>
-        <mesh filename="file:///home/halit/acrome_mini_robot/src/set_slam/meshes/left_wheel.stl" scale="1 1 1"/>
-      </geometry>
-    </collision>
-  </link>
-  <joint name="left_wheel_joint" type="continuous">
+      <origin xyz="0 0 0" rpy="0 0 0"/>
+      <inertia ixx="0.00045" ixy="0.0" ixz="0.0" iyy="0.00045" iyz="0.0" izz="0.00045"/>
+    </inertial>
+  </link>
+  <!-- Tekerlek 3 - Düzeltilmiş -->
+  <link name="wheel_3">
+    <visual>
+      <geometry>
+        <mesh filename="file:///home/halit/acrome_mini_robot/src/set_slam/meshes/right_wheel.stl" scale="0.7 0.7 0.7"/>
+      </geometry>
+      <origin xyz="0 0 0" rpy="1.5708 0 0"/>
+      <material name="black">
+        <color rgba="0.1 0.1 0.1 1"/>
+      </material>
+    </visual>
+    <collision>
+      <geometry>
+        <cylinder radius="0.06" length="0.025"/>
+      </geometry>
+      <origin xyz="0 0 0" rpy="1.5708 0 0"/>
+    </collision>
+    <inertial>
+      <mass value="0.25"/>
+      <origin xyz="0 0 0" rpy="0 0 0"/>
+      <inertia ixx="0.00045" ixy="0.0" ixz="0.0" iyy="0.00045" iyz="0.0" izz="0.00045"/>
+    </inertial>
+  </link>
+  <joint name="base_to_caster_support" type="fixed">
     <parent link="base_link"/>
-    <child link="left_wheel_link"/>
-    <!--
-      The wheel rotates around its axle; with REP-103 this is +Y.
-      Tune xyz to place the wheel correctly relative to the base mesh.
-      Example values below assume ~0.18 m track width and ~0.04 m radius.
-    -->
-    <origin xyz="-0.14 0 -0.01" rpy="0 0 0"/>
-    <axis xyz="0 1 0"/>
-  </joint>
-  <!-- ================ Right Wheel ================ -->
-  <link name="right_wheel_link">
-    <inertial>
-      <origin xyz="0 0 0" rpy="0 0 0"/>
-      <mass value="0.25"/>
-      <inertia ixx="0.0005" ixy="0.0" ixz="0.0" iyy="0.0007" iyz="0.0" izz="0.0005"/>
-    </inertial>
-    <visual>
-      <origin xyz="0 0 0" rpy="0 0 0"/>
-      <geometry>
-        <mesh filename="file:///home/halit/acrome_mini_robot/src/set_slam/meshes/right_wheel.stl" scale="1 1 1"/>
-      </geometry>
-      <material name="wheel_black"/>
-    </visual>
-    <collision>
-      <origin xyz="0 0 0" rpy="0 0 0"/>
-      <geometry>
-        <mesh filename="file:///home/halit/acrome_mini_robot/src/set_slam/meshes/right_wheel.stl" scale="1 1 1"/>
-      </geometry>
-    </collision>
-  </link>
-  <joint name="right_wheel_joint" type="continuous">
+    <child link="caster_support"/>
+    <origin xyz="0.085 0 0.05" rpy="0 0 0"/>
+  </joint>
+  <joint name="caster_support_to_wheel" type="continuous">
+    <parent link="caster_support"/>
+    <child link="caster_wheel"/>
+    <origin xyz="0 0 -0.03" rpy="0 0 0"/>
+    <axis xyz="0 0 1"/>
+    <dynamics damping="0.001" friction="0.001"/>
+  </joint>
+  <joint name="base_to_wheel_2" type="continuous">
     <parent link="base_link"/>
-    <child link="right_wheel_link"/>
-    <origin xyz="0.14 0 -0.01" rpy="0 0 0"/>
-    <axis xyz="0 1 0"/>
-  </joint>
-  <!-- ================= Optional caster (placeholder) ================= -->
-  <!-- If your robot has a caster, define it here and connect with a fixed joint. -->
-  <link name="caster_link">
-    <visual>
-      <geometry>
-        <cylinder radius="0.02" length="0.01"/>
-      </geometry>
-      <material name="caster_grey"><color rgba="0.5 0.5 0.5 1.0"/></material>
-    </visual>
-  </link>
-  <joint name="caster_joint" type="fixed">
+    <child link="wheel_2"/>
+    <origin xyz="0 0.13 0.045" rpy="0 0 -1.5708"/>
+    <axis xyz="1 0 0"/>
+    <dynamics damping="0.1" friction="0.01"/>
+  </joint>
+  <joint name="base_to_wheel_3" type="continuous">
     <parent link="base_link"/>
-    <child link="caster_link"/>
-    <origin xyz="-0.08 0 -0.02" rpy="0 0 0"/>
-  </joint>
-  <!-- ================= Coordinate frames (visual aids) ================= -->
-  <!-- Small axis markers to help verify orientation in RViz -->
-  <link name="base_axis_vis">
-    <visual>
-      <origin xyz="0 0 0" rpy="0 0 0"/>
-      <geometry>
-        <box size="0.001 0.001 0.001"/>
-      </geometry>
-      <material name="transparent"><color rgba="0 0 0 0"/></material>
-    </visual>
-  </link>
-  <joint name="base_axis_joint" type="fixed">
-    <parent link="base_link"/>
-    <child link="base_axis_vis"/>
-    <origin xyz="0 0 0" rpy="0 0 0"/>
-  </joint>
-  <!-- ================= Notes =================
-    * Tune the left/right wheel joint <origin> xyz until the wheels sit correctly in the model.
-    * For simulation or control, add transmissions and gazebo_ros2_control plugins separately.
-  ================= -->
+    <child link="wheel_3"/>
+    <origin xyz="0 -0.13 0.045" rpy="0 0 -1.5708"/>
+    <axis xyz="1 0 0"/>
+    <dynamics damping="0.1" friction="0.01"/>
+  </joint>
+  <!-- ROS2 Control -->
+  <ros2_control name="GazeboSimSystem" type="system">
+    <hardware>
+      <plugin>gz_ros2_control/GazeboSimSystem</plugin>
+    </hardware>
+    <joint name="base_to_wheel_2">
+      <command_interface name="velocity">
+        <param name="min">-10</param>
+        <param name="max">10</param>
+      </command_interface>
+      <state_interface name="position"/>
+      <state_interface name="velocity"/>
+      <state_interface name="effort"/>
+    </joint>
+    <joint name="base_to_wheel_3">
+      <command_interface name="velocity">
+        <param name="min">-10</param>
+        <param name="max">10</param>
+      </command_interface>
+      <state_interface name="position"/>
+      <state_interface name="velocity"/>
+      <state_interface name="effort"/>
+    </joint>
+    <!-- Caster wheel state yayınlamak için dummy joint -->
+    <joint name="caster_support_to_wheel">
+      <state_interface name="position"/>
+      <state_interface name="velocity"/>
+      <state_interface name="effort"/>
+    </joint>
+  </ros2_control>
+  <!-- Gazebo pluginleri -->
+  <gazebo>
+    <plugin filename="gz_ros2_control-system" name="gz_ros2_control::GazeboSimROS2ControlPlugin">
+      <parameters>$(find set_slam)/config/controllers_params.yaml</parameters>
+    </plugin>
+  </gazebo>
+  <!-- Ana gövde sürtünmesini düşür -->
+  <gazebo reference="base_link">
+    <mu1>0.1</mu1>
+    <mu2>0.1</mu2>
+    <material>Gazebo/Blue</material>
+  </gazebo>
+  <!-- Gazebo Caster Support Ayarları -->
+  <gazebo reference="caster_support">
+    <mu1>0.1</mu1>
+    <mu2>0.1</mu2>
+    <material>Gazebo/Grey</material>
+  </gazebo>
+  <!-- Gazebo Caster Wheel Ayarları -->
+  <gazebo reference="caster_wheel">
+    <!-- Düşük sürtünme - kolayca kayabilir -->
+    <mu1>0.1</mu1>
+    <mu2>0.1</mu2>
+    <!-- Düşük sertlik değerleri -->
+    <kp>2000.0</kp>
+    <kd>5.0</kd>
+    <minDepth>0.001</minDepth>
+    <maxVel>1.0</maxVel>
+    <material>Gazebo/Black</material>
+  </gazebo>
+  <gazebo reference="wheel_2">
+    <mu1>1.5</mu1>
+    <mu2>1.5</mu2>
+    <kp>2000.0</kp>
+    <kd>5.0</kd>
+    <minDepth>0.001</minDepth>
+    <maxVel>1.0</maxVel>
+    <material>Gazebo/Black</material>
+  </gazebo>
+  <gazebo reference="wheel_3">
+    <mu1>1.5</mu1>
+    <mu2>1.5</mu2>
+    <kp>2000.0</kp>
+    <kd>5.0</kd>
+    <minDepth>0.001</minDepth>
+    <maxVel>1.0</maxVel>
+    <material>Gazebo/Black</material>
+  </gazebo>
 </robot>

Commit message: gazebo controller is added, and robot's model is fixed

File: install/set_slam/share/set_slam/urdf/acrome_mini_robot.xacro (robot description, xacro)
@@ -1,7 +1,5 @@
 <?xml version="1.0"?>
 <robot name="acrome_mini_robot" xmlns:xacro="http://www.ros.org/wiki/xacro">
-  <!-- Parametreler -->
   <xacro:property name="PI" value="3.141592653589793"/>
-  <!-- Ana robot gövdesi -->
   <link name="base_link">
     <visual>
@@ -26,5 +24,4 @@
     </inertial>
   </link>
-  <!-- Caster Wheel Support (Destek Çubuğu) -->
   <link name="caster_support">
     <visual>
@@ -49,9 +46,8 @@
     </inertial>
   </link>
-  <!-- Caster Wheel -->
   <link name="caster_wheel">
     <visual>
       <geometry>
-        <sphere radius="0.02"/>
+        <sphere radius="0.01"/>
       </geometry>
       <origin xyz="0 0 0" rpy="0 0 0"/>
@@ -62,5 +58,5 @@
     <collision>
       <geometry>
-        <sphere radius="0.02"/>
+        <sphere radius="0.01"/>
       </geometry>
       <origin xyz="0 0 0" rpy="0 0 0"/>
@@ -72,9 +68,8 @@
     </inertial>
   </link>
-  <!-- Tekerlek 2 -->
   <link name="wheel_2">
     <visual>
       <geometry>
-        <mesh filename="file:///home/halit/acrome_mini_robot/src/set_slam/meshes/left_wheel.stl" scale="0.7 0.7 0.7"/>
+        <mesh filename="file:///home/halit/acrome_mini_robot/src/set_slam/meshes/left_wheel.stl" scale="0.36 0.36 0.36"/>
       </geometry>
       <origin xyz="0 0 0" rpy="1.5708 0 0"/>
@@ -93,19 +88,18 @@
       </surface>
       <geometry>
-        <cylinder radius="0.06" length="0.025"/>
-      </geometry>
-      <origin xyz="0 0 0" rpy="1.5708 0 0"/>
-    </collision>
-    <inertial>
-      <mass value="0.25"/>
-      <origin xyz="0 0 0" rpy="0 0 0"/>
-      <inertia ixx="0.00045" ixy="0.0" ixz="0.0" iyy="0.00045" iyz="0.0" izz="0.00045"/>
-    </inertial>
-  </link>
-  <!-- Tekerlek 3 - Düzeltilmiş -->
+        <cylinder radius="0.036" length="0.03"/>
+      </geometry>
+      <origin xyz="0 0 0" rpy="0 1.5708 0"/>
+    </collision>
+    <inertial>
+      <mass value="0.5"/>
+      <origin xyz="0 0 0" rpy="0 0 0"/>
+      <inertia ixx="0.001" ixy="0.0" ixz="0.0" iyy="0.001" iyz="0.0" izz="0.001"/>
+    </inertial>
+  </link>
   <link name="wheel_3">
     <visual>
       <geometry>
-        <mesh filename="file:///home/halit/acrome_mini_robot/src/set_slam/meshes/right_wheel.stl" scale="0.7 0.7 0.7"/>
+        <mesh filename="file:///home/halit/acrome_mini_robot/src/set_slam/meshes/right_wheel.stl" scale="0.36 0.36 0.36"/>
       </geometry>
       <origin xyz="0 0 0" rpy="1.5708 0 0"/>
@@ -115,13 +109,21 @@
     </visual>
     <collision>
-      <geometry>
-        <cylinder radius="0.06" length="0.025"/>
-      </geometry>
-      <origin xyz="0 0 0" rpy="1.5708 0 0"/>
-    </collision>
-    <inertial>
-      <mass value="0.25"/>
-      <origin xyz="0 0 0" rpy="0 0 0"/>
-      <inertia ixx="0.00045" ixy="0.0" ixz="0.0" iyy="0.00045" iyz="0.0" izz="0.00045"/>
+      <surface>
+        <friction>
+          <ode>
+            <mu>1.0</mu>
+            <mu2>1.0</mu2>
+          </ode>
+        </friction>
+      </surface>
+      <geometry>
+        <cylinder radius="0.036" length="0.03"/>
+      </geometry>
+      <origin xyz="0 0 0" rpy="0 1.5708 0"/>
+    </collision>
+    <inertial>
+      <mass value="0.5"/>
+      <origin xyz="0 0 0" rpy="0 0 0"/>
+      <inertia ixx="0.001" ixy="0.0" ixz="0.0" iyy="0.001" iyz="0.0" izz="0.001"/>
     </inertial>
   </link>
@@ -129,5 +131,5 @@
     <parent link="base_link"/>
     <child link="caster_support"/>
-    <origin xyz="0.085 0 0.05" rpy="0 0 0"/>
+    <origin xyz="0.085 0 0.04" rpy="0 0 0"/>
   </joint>
   <joint name="caster_support_to_wheel" type="continuous">
@@ -141,5 +143,5 @@
     <parent link="base_link"/>
     <child link="wheel_2"/>
-    <origin xyz="0 0.13 0.045" rpy="0 0 -1.5708"/>
+    <origin xyz="0 0.129 0.025" rpy="0 0 -1.5708"/>
     <axis xyz="1 0 0"/>
     <dynamics damping="0.1" friction="0.01"/>
@@ -148,9 +150,8 @@
     <parent link="base_link"/>
     <child link="wheel_3"/>
-    <origin xyz="0 -0.13 0.045" rpy="0 0 -1.5708"/>
+    <origin xyz="0 -0.129 0.025" rpy="0 0 -1.5708"/>
     <axis xyz="1 0 0"/>
     <dynamics damping="0.1" friction="0.01"/>
   </joint>
-  <!-- ROS2 Control -->
   <ros2_control name="GazeboSimSystem" type="system">
     <hardware>
@@ -175,5 +176,4 @@
       <state_interface name="effort"/>
     </joint>
-    <!-- Caster wheel state yayınlamak için dummy joint -->
     <joint name="caster_support_to_wheel">
       <state_interface name="position"/>
@@ -182,5 +182,4 @@
     </joint>
   </ros2_control>
-  <!-- Gazebo pluginleri -->
   <gazebo>
     <plugin filename="gz_ros2_control-system" name="gz_ros2_control::GazeboSimROS2ControlPlugin">
@@ -188,5 +187,4 @@
     </plugin>
   </gazebo>
-  <!-- Ana gövde sürtünmesini düşür -->
   <gazebo reference="base_link">
     <mu1>0.1</mu1>
@@ -194,5 +192,4 @@
     <material>Gazebo/Blue</material>
   </gazebo>
-  <!-- Gazebo Caster Support Ayarları -->
   <gazebo reference="caster_support">
     <mu1>0.1</mu1>
@@ -200,10 +197,7 @@
     <material>Gazebo/Grey</material>
   </gazebo>
-  <!-- Gazebo Caster Wheel Ayarları -->
   <gazebo reference="caster_wheel">
-    <!-- Düşük sürtünme - kolayca kayabilir -->
     <mu1>0.1</mu1>
     <mu2>0.1</mu2>
-    <!-- Düşük sertlik değerleri -->
     <kp>2000.0</kp>
     <kd>5.0</kd>
@@ -213,8 +207,8 @@
   </gazebo>
   <gazebo reference="wheel_2">
-    <mu1>1.5</mu1>
-    <mu2>1.5</mu2>
-    <kp>2000.0</kp>
-    <kd>5.0</kd>
+    <mu1>1.0</mu1>
+    <mu2>1.0</mu2>
+    <kp>1000000.0</kp>
+    <kd>100.0</kd>
     <minDepth>0.001</minDepth>
     <maxVel>1.0</maxVel>
@@ -222,8 +216,8 @@
   </gazebo>
   <gazebo reference="wheel_3">
-    <mu1>1.5</mu1>
-    <mu2>1.5</mu2>
-    <kp>2000.0</kp>
-    <kd>5.0</kd>
+    <mu1>1.0</mu1>
+    <mu2>1.0</mu2>
+    <kp>1000000.0</kp>
+    <kd>100.0</kd>
     <minDepth>0.001</minDepth>
     <maxVel>1.0</maxVel>

Commit message: imu plugin is removed

File: install/set_slam/share/set_slam/urdf/acrome_mini_robot.xacro (robot description, xacro)
@@ -51,79 +51,4 @@
     <origin xyz="0 0 0.175" rpy="0 0 0"/>
   </joint>
-  <link name="imu_link">
-    <visual>
-      <geometry>
-        <box size="0.02 0.02 0.02"/>
-      </geometry>
-      <material name="red">
-        <color rgba="1.0 0.0 0.0 1.0"/>
-      </material>
-    </visual>
-    <collision>
-      <geometry>
-        <box size="0.02 0.02 0.02"/>
-      </geometry>
-    </collision>
-    <inertial>
-      <mass value="0.01"/>
-      <inertia ixx="0.00001" ixy="0" ixz="0" iyy="0.00001" iyz="0" izz="0.00001"/>
-    </inertial>
-  </link>
-  <joint name="imu_joint" type="fixed">
-    <parent link="base_link"/>
-    <child link="imu_link"/>
-    <origin xyz="0 0 0.075" rpy="0 0 0"/> </joint>
-  <gazebo reference="imu_link">
-    <sensor name="imu" type="imu">
-      <always_on>true</always_on>
-      <update_rate>100</update_rate>
-      <visualize>true</visualize>
-      <topic>imu</topic>
-      <gz_frame_id>imu_link</gz_frame_id>
-      <frame_id>imu_link</frame_id>
-      <imu>
-        <angular_velocity>
-          <x>
-            <noise type="gaussian">
-              <mean>0.0</mean>
-              <stddev>2e-4</stddev>
-            </noise>
-          </x>
-          <y>
-            <noise type="gaussian">
-              <mean>0.0</mean>
-              <stddev>2e-4</stddev>
-            </noise>
-          </y>
-          <z>
-            <noise type="gaussian">
-              <mean>0.0</mean>
-              <stddev>2e-4</stddev>
-            </noise>
-          </z>
-        </angular_velocity>
-        <linear_acceleration>
-          <x>
-            <noise type="gaussian">
-              <mean>0.0</mean>
-              <stddev>1.7e-2</stddev>
-            </noise>
-          </x>
-          <y>
-            <noise type="gaussian">
-              <mean>0.0</mean>
-              <stddev>1.7e-2</stddev>
-            </noise>
-          </y>
-          <z>
-            <noise type="gaussian">
-              <mean>0.0</mean>
-              <stddev>1.7e-2</stddev>
-            </noise>
-          </z>
-        </linear_acceleration>
-      </imu>
-      </sensor>
-  </gazebo>
   <link name="caster_support">
     <visual>
